Commit message: wheels controlled with python

File: my_robot/my_robot/urdf/my_robot.urdf.xacro (robot description, xacro)
@@ -13,5 +13,4 @@
     </inertial>
   </xacro:macro>
-  <link name="world"/>
 <!--
   <link name="my_robot_xpart">
@@ -54,4 +53,19 @@
   </transmission>
 -->
+<link name="base_footprint">
+  <visual>
+    <origin rpy="0 0 0" xyz="0 0 0"/>
+    <geometry>
+      <box size="0 0 0"/>
+    </geometry>
+  </visual>
+  <collision>
+    <origin rpy="0 0 0" xyz="0 0 0"/>
+    <geometry>
+      <box size="0 0 0"/>
+    </geometry>
+  </collision>
+  <xacro:default_inertial mass="0.1"/>
+</link>
   <link name="base_link">
     <visual>
@@ -67,5 +81,5 @@
       </geometry>
     </collision>
-    <xacro:default_inertial mass="0.1"/>
+    <xacro:default_inertial mass="10"/>
   </link>
   <link name="wheel_1">
@@ -84,5 +98,5 @@
         </geometry>
     </collision>
-    <xacro:default_inertial mass="0.1"/>
+    <xacro:default_inertial mass="3"/>
 </link>
 <link name="wheel_2">
@@ -101,63 +115,63 @@
       </geometry>
   </collision>
+  <xacro:default_inertial mass="3"/>
+</link>
+<link name="wheel_3">
+  <visual>
+          <geometry>
+              <cylinder length="${length_wheel}" radius="${radius_wheel}"/>
+          </geometry>
+      <origin rpy="0 0 0" xyz="0 0 0"/>
+      <material name="black">
+          <color rgba="0 0 0 1"/>
+      </material>
+  </visual>
+  <collision>
+      <geometry>
+              <cylinder length="${length_wheel}" radius="${radius_wheel}"/>
+      </geometry>
+  </collision>
+  <xacro:default_inertial mass="3"/>
+</link>
+<link name="wheel_4">
+  <visual>
+          <geometry>
+              <cylinder length="${length_wheel}" radius="${radius_wheel}"/>
+          </geometry>
+      <origin rpy="0 0 0" xyz="0 0 0"/>
+      <material name="black">
+          <color rgba="0 0 0 1"/>
+      </material>
+  </visual>
+  <collision>
+      <geometry>
+              <cylinder length="${length_wheel}" radius="${radius_wheel}"/>
+      </geometry>
+  </collision>
+  <xacro:default_inertial mass="3"/>
+</link>
+<link name="imu_link">
+  <visual>
+    <geometry>
+      <box size="0.1 0.1 0.1"/>
+    </geometry>
+    <origin rpy="0 0 0" xyz="0 0 0"/>
+    <material name="black">
+          <color rgba="0 0 0 1"/>
+    </material>
+  </visual>
+  <collision>
+    <geometry>
+      <box size="0.1 0.1 0.1"/>
+    </geometry>
+  </collision>
   <xacro:default_inertial mass="0.1"/>
 </link>
-<link name="wheel_3">
-  <visual>
-      <geometry>
-          <cylinder length="${length_wheel}" radius="${radius_wheel}"/>
-      </geometry>
-      <origin rpy="0 0 0" xyz="0 0 0"/>
-      <material name="black">
-          <color rgba="0 0 0 1"/>
-      </material>
-  </visual>
-  <collision>
-      <geometry>
-              <cylinder length="${length_wheel}" radius="${radius_wheel}"/>
-      </geometry>
-  </collision>
-  <xacro:default_inertial mass="0.1"/>
-</link>
-<link name="wheel_4">
-  <visual>
-          <geometry>
-              <cylinder length="${length_wheel}" radius="${radius_wheel}"/>
-          </geometry>
-      <origin rpy="0 0 0" xyz="0 0 0"/>
-      <material name="black">
-          <color rgba="0 0 0 1"/>
-      </material>
-  </visual>
-  <collision>
-      <geometry>
-              <cylinder length="${length_wheel}" radius="${radius_wheel}"/>
-      </geometry>
-  </collision>
-  <xacro:default_inertial mass="0.1"/>
-</link>
-<link name="imu_link">
-  <visual>
-    <geometry>
-      <box size="0.1 0.1 0.1"/>
-    </geometry>
-    <origin rpy="0 0 0" xyz="0 0 0"/>
-    <material name="black">
-          <color rgba="0 0 0 1"/>
-    </material>
-  </visual>
-  <collision>
-    <geometry>
-      <box size="0.1 0.1 0.1"/>
-    </geometry>
-  </collision>
-  <xacro:default_inertial mass="0.1"/>
-</link>
   <joint name="my_robot_base" type="prismatic">
     <origin rpy="0 0 0" xyz="0 0 0"/>
-    <parent link="world"/>
+    <parent link="base_footprint"/>
     <child link="base_link"/>
     <axis xyz="0 1 0"/>
-    <dynamics damping="0" friction="0"/>
+    <dynamics damping="1" friction="1"/>
     <limit effort="10000" lower="-50.0" upper="600.0" velocity="0.1"/>
   </joint>
@@ -165,5 +179,5 @@
     <parent link="base_link"/>
     <child link="wheel_1"/>
-    <origin rpy="0 1.5707 0" xyz="0.6 0.4 0"/>
+    <origin rpy="0 -1.5707 0" xyz="0.6 0.4 0"/>
     <axis xyz="0 0 1" />
   </joint>
@@ -171,5 +185,5 @@
     <parent link="base_link"/>
     <child link="wheel_2"/>
-    <origin rpy="0 1.5707 0" xyz="-0.6 0.4 0"/>
+    <origin rpy="0 -1.5707 0" xyz="-0.6 0.4 0"/>
     <axis xyz="0 0 1" />
   </joint>
@@ -177,5 +191,5 @@
     <parent link="base_link"/>
     <child link="wheel_3"/>
-    <origin rpy="0 1.5707 0" xyz="0.6 -0.4 0"/>
+    <origin rpy="0 -1.5707 0" xyz="0.6 -0.4 0"/>
     <axis xyz="0 0 1" />
   </joint>
@@ -183,5 +197,5 @@
     <parent link="base_link"/>
     <child link="wheel_4"/>
-    <origin rpy="0 1.5707 0" xyz="-0.6 -0.4 0"/>
+    <origin rpy="0 -1.5707 0" xyz="-0.6 -0.4 0"/>
     <axis xyz="0 0 1" />
   </joint>
@@ -202,4 +216,24 @@
     </actuator>
   </transmission>
+  <transmission name="transmission_wheel_1">
+    <type>transmission_interface/SimpleTransmission</type>
+    <joint name="base_to_wheel1">
+        <hardwareInterface>hardware_interface/EffortJointInterface</hardwareInterface>
+    </joint>
+    <actuator name="motor_wheel_1">
+        <hardwareInterface>hardware_interface/EffortJointInterface</hardwareInterface>
+        <mechanicalReduction>1</mechanicalReduction>
+    </actuator>
+</transmission>
+<transmission name="transmission_wheel_2">
+  <type>transmission_interface/SimpleTransmission</type>
+  <joint name="base_to_wheel2">
+      <hardwareInterface>hardware_interface/EffortJointInterface</hardwareInterface>
+  </joint>
+  <actuator name="motor_wheel_2">
+      <hardwareInterface>hardware_interface/EffortJointInterface</hardwareInterface>
+      <mechanicalReduction>1</mechanicalReduction>
+  </actuator>
+</transmission>
 <!--
   <joint name="entity" type="fixed">
@@ -210,4 +244,5 @@
 <gazebo reference="base_link">
     <material>Gazebo/Blue</material>
+    <gravity>1</gravity>
 </gazebo>
 <gazebo reference="wheel_1">
