Commit message: add python script

File: my_robot/urdf/my_robot.urdf.xacro (robot description, xacro)
@@ -1,45 +1,42 @@
 <?xml version="1.0"?>
 <robot xmlns:xacro="http://www.ros.org/wiki/xacro" name="my_robot">
-  <xacro:property name="length" value="2" />
+  <xacro:property name="length" value="1" />
   <xacro:property name="width" value="1" />
   <xacro:property name="height" value="0.5" />
-  <material name="blue">
-  <color rgba="1 0 0.8 1"/>
-  </material>
   <xacro:macro name="default_inertial" params="mass">
     <inertial>
       <origin rpy="0.0 0 0" xyz="0 0 0"/>
       <mass value="${mass}" />
-      <inertia ixx="1.0" ixy="0.0" ixz="0.0" iyy="1.0" iyz="0.0" izz="1.0" />
+      <inertia ixx="0.4" ixy="0.0" ixz="0.0" iyy="0.4" iyz="0.0" izz="0.2" />
     </inertial>
   </xacro:macro>
   <link name="world"/>
-  <link name="my_robot_link">
+  <link name="my_robot_xpart">
     <visual>
-      <origin rpy="0 0 0" xyz="0 0 0"/>
+      <origin rpy="0 0 0" xyz="0 0 ${height/2}"/>
       <geometry>
-        <box size="${length} ${width} ${height}"/>
+        <box size="${length} ${width} ${height/2}"/>
       </geometry>
-      <material name="blue"/>
     </visual>
     <collision>
-      <origin rpy="0 0 0" xyz="0 0 0"/>
+      <origin rpy="0 0 0" xyz="0 0 ${height/2}"/>
       <geometry>
-        <box size="${length} ${width} ${height}"/>
+        <box size="${length} ${width} ${height/2}"/>
       </geometry>
     </collision>
     <xacro:default_inertial mass="10"/>
   </link>
-  <gazebo reference="my_robot_link">
+  <gazebo reference="my_robot_xpart">
     <mu1>10.0</mu1>
     <mu2>10.0</mu2>
-    <material> Gazebo/Red</material>
+    <material> Gazebo/GreyTransparent</material>
   </gazebo>
   <joint name="my_robot_x" type="prismatic">
     <origin rpy="0 0 0" xyz="0 0 0"/>
     <parent link="world"/>
-    <child link="my_robot_link"/>
+    <child link="my_robot_xpart"/>
     <axis xyz="1 0 0"/>
-    <limit effort="10000" lower="-5.0" upper="5.0" velocity="1"/>
+    <dynamics damping="0" friction="0"/>
+    <limit effort="10000" lower="-50.0" upper="50.0" velocity="1"/>
   </joint>
   <transmission name="tran1">
@@ -53,4 +50,48 @@
     </actuator>
   </transmission>
+  <link name="my_robot_ypart">
+    <visual>
+      <origin rpy="0 0 0" xyz="0 0 0"/>
+      <geometry>
+        <box size="${length} ${width} ${height/2}"/>
+      </geometry>
+    </visual>
+    <collision>
+      <origin rpy="0 0 0" xyz="0 0 0"/>
+      <geometry>
+        <box size="${length} ${width} ${height/2}"/>
+      </geometry>
+    </collision>
+    <xacro:default_inertial mass="10"/>
+  </link>
+  <gazebo reference="my_robot_ypart">
+    <mu1>10.0</mu1>
+    <mu2>10.0</mu2>
+    <material> Gazebo/Blue</material>
+  </gazebo>
+  <joint name="my_robot_y" type="prismatic">
+    <origin rpy="0 0 0" xyz="0 0 0"/>
+    <parent link="my_robot_xpart"/>
+    <child link="my_robot_ypart"/>
+    <axis xyz="0 1 0"/>
+    <dynamics damping="0" friction="0"/>
+    <limit effort="10000" lower="-50.0" upper="50.0" velocity="1"/>
+  </joint>
+  <transmission name="tran2">
+    <type>transmission_interface/SimpleTransmission</type>
+    <joint name="my_robot_y">
+      <hardwareInterface>EffortJointInterface</hardwareInterface>
+    </joint>
+    <actuator name="motor2">
+      <hardwareInterface>EffortJointInterface</hardwareInterface>
+      <mechanicalReduction>1</mechanicalReduction>
+    </actuator>
+  </transmission>
+<!--
+  <joint name="entity" type="fixed">
+    <origin rpy="0 0 0" xyz="0 0 0"/>
+    <parent link="my_robot_xpart"/>
+    <child link="my_robot_ypart"/>
+  </joint>-->
   <!-- Gazebo plugin for ROS Control -->
   <gazebo>

Commit message: Add files via upload

File: my_robot/urdf/my_robot.urdf.xacro (robot description, xacro)
@@ -4,4 +4,9 @@
   <xacro:property name="width" value="1" />
   <xacro:property name="height" value="0.5" />
+  <xacro:property name="imu_link" value="0.1" /> <!-- Size of imu -->
+  <xacro:property name="hokuyo_link" value="0.1" /> <!-- Size of hokuyo -->
+  <xacro:property name="camera_link" value="0.1" /> <!-- Size of camera -->
+<!-- Import all Gazebo-customization elements, including Gazebo colors -->
+  <xacro:include filename="$(find my_robot)/urdf/my_robot.gazebo" />
   <material name="blue">
   <color rgba="1 0 0.8 1"/>
@@ -54,8 +59,97 @@
   </transmission>
   <!-- Gazebo plugin for ROS Control -->
-  <gazebo>
+    <gazebo>
     <plugin name="gazebo_ros_control" filename="libgazebo_ros_control.so">
       <robotNamespace>/my_robot</robotNamespace>
     </plugin>
   </gazebo>
+   <!-- Gazebo plugin for imu -->
+  <joint name="imu_joint" type="fixed">
+    <axis xyz="0 0 0" />
+    <origin xyz="${length/2+imu_link/2} 0 0" rpy="0 0 0"/>
+    <parent link="my_robot_link"/>
+    <child link="imu_link"/>
+  </joint>
+    <link name="imu_link">
+    <collision>
+      <origin xyz="0 0 0" rpy="0 0 0"/>
+      <geometry>
+	<box size="${imu_link} ${imu_link} ${imu_link}"/>
+      </geometry>
+    </collision>
+    <visual>
+      <origin xyz="0 0 0" rpy="0 0 0"/>
+      <geometry>
+        <box size="${imu_link} ${imu_link} ${imu_link}"/>
+      </geometry>
+    </visual>
+    <inertial>
+      <mass value="1e-5" />
+      <origin xyz="0 0 0" rpy="0 0 0"/>
+      <inertia ixx="1e-6" ixy="0" ixz="0" iyy="1e-6" iyz="0" izz="1e-6" />
+    </inertial>
+  </link>
+  <!-- Gazebo plugin for laser scan sensor -->
+  <joint name="hokuyo_joint" type="fixed">
+    <axis xyz="0 0 0" />
+    <origin xyz="0 ${-width/2-hokuyo_link/2} 0" rpy="0 0 0"/>
+    <parent link="my_robot_link"/>
+    <child link="hokuyo_link"/>
+  </joint>
+  <link name="hokuyo_link">
+    <collision>
+      <origin xyz="0 0 0" rpy="0 0 0"/>
+      <geometry>
+	<box size="0.1 0.1 0.1"/>
+      </geometry>
+    </collision>
+    <visual>
+      <origin xyz="0 0 0" rpy="0 0 0"/>
+      <geometry>
+        <box size="${hokuyo_link} ${hokuyo_link} ${hokuyo_link}"/>
+      </geometry>
+    </visual>
+    <inertial>
+      <mass value="1e-5" />
+      <origin xyz="0 0 0" rpy="0 0 0"/>
+      <inertia ixx="1e-6" ixy="0" ixz="0" iyy="1e-6" iyz="0" izz="1e-6" />
+    </inertial>
+  </link>
+  <!-- Camera -->
+  <joint name="camera_joint" type="fixed">
+    <axis xyz="0 0 0" />
+    <origin xyz="0 0 ${height/2+camera_link/2} " rpy="0 0 0"/>
+    <parent link="my_robot_link"/>
+    <child link="camera_link"/>
+  </joint>
+  <link name="camera_link">
+    <collision>
+      <origin xyz="0 0 0" rpy="0 0 0"/>
+      <geometry>
+	<box size="${camera_link} ${camera_link} ${camera_link}"/>
+      </geometry>
+    </collision>
+    <visual>
+      <origin xyz="0 0 0" rpy="0 0 0"/>
+      <geometry>
+	<box size="${camera_link} ${camera_link} ${camera_link}"/>
+      </geometry>
+    </visual>
+    <inertial>
+      <mass value="1e-5" />
+      <origin xyz="0 0 0" rpy="0 0 0"/>
+      <inertia ixx="1e-6" ixy="0" ixz="0" iyy="1e-6" iyz="0" izz="1e-6" />
+    </inertial>
+  </link>
+    <!-- generate an optical frame http://www.ros.org/reps/rep-0103.html#suffix-frames
+      so that ros and opencv can operate on the camera frame correctly -->
+  <joint name="camera_optical_joint" type="fixed">
+    <!-- these values have to be these values otherwise the gazebo camera image
+        won't be aligned properly with the frame it is supposedly originating from -->
+    <origin xyz="0 0 0" rpy="${-pi/2} 0 ${-pi/2}"/>
+    <parent link="camera_link"/>
+    <child link="camera_link_optical"/>
+  </joint>
+  <link name="camera_link_optical">
+  </link>
 </robot>

Commit message: ready to merge

File: my_robot/urdf/my_robot.urdf.xacro (robot description, xacro)
@@ -8,8 +8,9 @@
       <origin rpy="0.0 0 0" xyz="0 0 0"/>
       <mass value="${mass}" />
-      <inertia ixx="0.4" ixy="0.0" ixz="0.0" iyy="0.4" iyz="0.0" izz="0.2" />
+      <inertia ixx="0.0" ixy="0.0" ixz="0.0" iyy="0.0" iyz="0.0" izz="0.0" />
     </inertial>
   </xacro:macro>
   <link name="world"/>
+<!--
   <link name="my_robot_xpart">
     <visual>
@@ -50,4 +51,5 @@
     </actuator>
   </transmission>
+-->
   <link name="my_robot_ypart">
     <visual>
@@ -63,5 +65,5 @@
       </geometry>
     </collision>
-    <xacro:default_inertial mass="10"/>
+    <xacro:default_inertial mass="0.1"/>
   </link>
   <gazebo reference="my_robot_ypart">
@@ -72,5 +74,5 @@
   <joint name="my_robot_y" type="prismatic">
     <origin rpy="0 0 0" xyz="0 0 0"/>
-    <parent link="my_robot_xpart"/>
+    <parent link="world"/>
     <child link="my_robot_ypart"/>
     <axis xyz="0 1 0"/>

Commit message: new world

File: my_robot/urdf/my_robot.urdf.xacro (robot description, xacro)
@@ -8,5 +8,5 @@
       <origin rpy="0.0 0 0" xyz="0 0 0"/>
       <mass value="${mass}" />
-      <inertia ixx="0.4" ixy="0.0" ixz="0.0" iyy="0.4" iyz="0.0" izz="0.2" />
+      <inertia ixx="0.0" ixy="0.0" ixz="0.0" iyy="0.0" iyz="0.0" izz="0.0" />
     </inertial>
   </xacro:macro>
@@ -25,5 +25,5 @@
       </geometry>
     </collision>
-    <xacro:default_inertial mass="10"/>
+    <xacro:default_inertial mass="1"/>
   </link>
   <gazebo reference="my_robot_xpart">
@@ -63,5 +63,5 @@
       </geometry>
     </collision>
-    <xacro:default_inertial mass="10"/>
+    <xacro:default_inertial mass="1"/>
   </link>
   <gazebo reference="my_robot_ypart">

Commit message: change max y position

File: my_robot/urdf/my_robot.urdf.xacro (robot description, xacro)
@@ -78,5 +78,5 @@
     <axis xyz="0 1 0"/>
     <dynamics damping="0" friction="0"/>
-    <limit effort="10000" lower="-50.0" upper="50.0" velocity="1"/>
+    <limit effort="10000" lower="-50.0" upper="600.0" velocity="1"/>
   </joint>
   <transmission name="tran2">

Commit message: added some stylish wheels ;)

File: my_robot/urdf/my_robot.urdf.xacro (robot description, xacro)
@@ -4,4 +4,6 @@
   <xacro:property name="width" value="1" />
   <xacro:property name="height" value="0.5" />
+  <xacro:property name="length_wheel" value="0.2" />
+  <xacro:property name="radius_wheel" value="0.2" />
   <xacro:macro name="default_inertial" params="mass">
     <inertial>
@@ -52,5 +54,5 @@
   </transmission>
 -->
-  <link name="my_robot_ypart">
+  <link name="base_link">
     <visual>
       <origin rpy="0 0 0" xyz="0 0 0"/>
@@ -67,20 +69,107 @@
     <xacro:default_inertial mass="0.1"/>
   </link>
-  <gazebo reference="my_robot_ypart">
-    <mu1>10.0</mu1>
-    <mu2>10.0</mu2>
-    <material> Gazebo/Blue</material>
-  </gazebo>
-  <joint name="my_robot_y" type="prismatic">
+  <link name="wheel_1">
+    <visual>
+            <geometry>
+                <cylinder length="${length_wheel}" radius="${radius_wheel}"/>
+            </geometry>
+        <origin rpy="0 0 0" xyz="0 0 0"/>
+        <material name="black">
+            <color rgba="0 0 0 1"/>
+        </material>
+    </visual>
+    <collision>
+        <geometry>
+                <cylinder length="${length_wheel}" radius="${radius_wheel}"/>
+        </geometry>
+    </collision>
+    <xacro:default_inertial mass="0.1"/>
+</link>
+<link name="wheel_2">
+  <visual>
+          <geometry>
+              <cylinder length="${length_wheel}" radius="${radius_wheel}"/>
+          </geometry>
+      <origin rpy="0 0 0" xyz="0 0 0"/>
+      <material name="black">
+          <color rgba="0 0 0 1"/>
+      </material>
+  </visual>
+  <collision>
+      <geometry>
+              <cylinder length="${length_wheel}" radius="${radius_wheel}"/>
+      </geometry>
+  </collision>
+  <xacro:default_inertial mass="0.1"/>
+</link>
+<link name="wheel_3">
+  <visual>
+          <geometry>
+              <cylinder length="${length_wheel}" radius="${radius_wheel}"/>
+          </geometry>
+      <origin rpy="0 0 0" xyz="0 0 0"/>
+      <material name="black">
+          <color rgba="0 0 0 1"/>
+      </material>
+  </visual>
+  <collision>
+      <geometry>
+              <cylinder length="${length_wheel}" radius="${radius_wheel}"/>
+      </geometry>
+  </collision>
+  <xacro:default_inertial mass="0.1"/>
+</link>
+<link name="wheel_4">
+  <visual>
+          <geometry>
+              <cylinder length="${length_wheel}" radius="${radius_wheel}"/>
+          </geometry>
+      <origin rpy="0 0 0" xyz="0 0 0"/>
+      <material name="black">
+          <color rgba="0 0 0 1"/>
+      </material>
+  </visual>
+  <collision>
+      <geometry>
+              <cylinder length="${length_wheel}" radius="${radius_wheel}"/>
+      </geometry>
+  </collision>
+  <xacro:default_inertial mass="0.1"/>
+</link>
+  <joint name="my_robot_base" type="prismatic">
     <origin rpy="0 0 0" xyz="0 0 0"/>
     <parent link="world"/>
-    <child link="my_robot_ypart"/>
+    <child link="base_link"/>
     <axis xyz="0 1 0"/>
     <dynamics damping="0" friction="0"/>
-    <limit effort="10000" lower="-50.0" upper="600.0" velocity="1"/>
+    <limit effort="10000" lower="-50.0" upper="600.0" velocity="0.1"/>
+  </joint>
+  <joint name="base_to_wheel1" type="continuous">
+    <parent link="base_link"/>
+    <child link="wheel_1"/>
+    <origin rpy="0 1.5707 0" xyz="0.6 0.4 0"/>
+    <axis xyz="0 0 1" />
+  </joint>
+  <joint name="base_to_wheel2" type="continuous">
+    <parent link="base_link"/>
+    <child link="wheel_2"/>
+    <origin rpy="0 1.5707 0" xyz="-0.6 0.4 0"/>
+    <axis xyz="0 0 1" />
+  </joint>
+  <joint name="base_to_wheel3" type="continuous">
+    <parent link="base_link"/>
+    <child link="wheel_3"/>
+    <origin rpy="0 1.5707 0" xyz="0.6 -0.4 0"/>
+    <axis xyz="0 0 1" />
+  </joint>
+  <joint name="base_to_wheel4" type="continuous">
+    <parent link="base_link"/>
+    <child link="wheel_4"/>
+    <origin rpy="0 1.5707 0" xyz="-0.6 -0.4 0"/>
+    <axis xyz="0 0 1" />
   </joint>
   <transmission name="tran2">
     <type>transmission_interface/SimpleTransmission</type>
-    <joint name="my_robot_y">
+    <joint name="my_robot_base">
       <hardwareInterface>EffortJointInterface</hardwareInterface>
     </joint>
@@ -96,4 +185,19 @@
     <child link="my_robot_ypart"/>
   </joint>-->
+<gazebo reference="base_link">
+    <material>Gazebo/Blue</material>
+</gazebo>
+<gazebo reference="wheel_1">
+    <material>Gazebo/Black</material>
+</gazebo>
+<gazebo reference="wheel_2">
+    <material>Gazebo/Black</material>
+</gazebo>
+<gazebo reference="wheel_3">
+    <material>Gazebo/Black</material>
+</gazebo>
+<gazebo reference="wheel_4">
+    <material>Gazebo/Black</material>
+</gazebo>
   <!-- Gazebo plugin for ROS Control -->
   <gazebo>

Commit message: Added an IMU sensor to the robot - topic: /imu

File: my_robot/urdf/my_robot.urdf.xacro (robot description, xacro)
@@ -105,4 +105,21 @@
 <link name="wheel_3">
   <visual>
+      <geometry>
+          <cylinder length="${length_wheel}" radius="${radius_wheel}"/>
+      </geometry>
+      <origin rpy="0 0 0" xyz="0 0 0"/>
+      <material name="black">
+          <color rgba="0 0 0 1"/>
+      </material>
+  </visual>
+  <collision>
+      <geometry>
+              <cylinder length="${length_wheel}" radius="${radius_wheel}"/>
+      </geometry>
+  </collision>
+  <xacro:default_inertial mass="0.1"/>
+</link>
+<link name="wheel_4">
+  <visual>
           <geometry>
               <cylinder length="${length_wheel}" radius="${radius_wheel}"/>
@@ -120,18 +137,18 @@
   <xacro:default_inertial mass="0.1"/>
 </link>
-<link name="wheel_4">
-  <visual>
-          <geometry>
-              <cylinder length="${length_wheel}" radius="${radius_wheel}"/>
-          </geometry>
-      <origin rpy="0 0 0" xyz="0 0 0"/>
-      <material name="black">
-          <color rgba="0 0 0 1"/>
-      </material>
-  </visual>
-  <collision>
-      <geometry>
-              <cylinder length="${length_wheel}" radius="${radius_wheel}"/>
-      </geometry>
+<link name="imu_link">
+  <visual>
+    <geometry>
+      <box size="0.1 0.1 0.1"/>
+    </geometry>
+    <origin rpy="0 0 0" xyz="0 0 0"/>
+    <material name="black">
+          <color rgba="0 0 0 1"/>
+    </material>
+  </visual>
+  <collision>
+    <geometry>
+      <box size="0.1 0.1 0.1"/>
+    </geometry>
   </collision>
   <xacro:default_inertial mass="0.1"/>
@@ -167,4 +184,10 @@
     <child link="wheel_4"/>
     <origin rpy="0 1.5707 0" xyz="-0.6 -0.4 0"/>
+    <axis xyz="0 0 1" />
+  </joint>
+  <joint name="base_to_imu" type="continuous">
+    <parent link="base_link"/>
+    <child link="imu_link"/>
+    <origin rpy="0.0 0.0 0.0" xyz="0.0 0.0 0.175"/>
     <axis xyz="0 0 1" />
   </joint>
@@ -206,3 +229,25 @@
     </plugin>
   </gazebo>
+  <!-- Gazebo plugin for IMU-->
+  <gazebo reference="imu_link">
+    <material>Gazebo/Black</material>
+    <gravity>true</gravity>
+    <sensor name="imu_sensor" type="imu">
+      <always_on>true</always_on>
+      <update_rate>100</update_rate>
+      <visualize>true</visualize>
+      <topic>__default_topic__</topic>
+      <plugin filename="libgazebo_ros_imu_sensor.so" name="imu_plugin">
+        <topicName>imu</topicName>
+        <bodyName>imu_link</bodyName>
+        <updateRateHZ>10.0</updateRateHZ>
+        <gaussianNoise>0.0</gaussianNoise>
+        <xyzOffset>0 0 0</xyzOffset>
+        <rpyOffset>0 0 0</rpyOffset>
+        <frameName>imu_link</frameName>
+        <initialOrientationAsReference>false</initialOrientationAsReference>
+      </plugin>
+      <pose>0 0 0 0 0 0</pose>
+    </sensor>
+  </gazebo>
 </robot>

Commit message: wheel properties update

File: my_robot/urdf/my_robot.urdf.xacro (robot description, xacro)
@@ -247,15 +247,30 @@
 </gazebo>
 <gazebo reference="wheel_1">
-    <material>Gazebo/Black</material>
+  <mu1 value="200.0"/>
+  <mu2 value="100.0"/>
+  <kp value="10000000.0" />
+  <kd value="1.0" />
+  <material>Gazebo/Grey</material>
 </gazebo>
 <gazebo reference="wheel_2">
-    <material>Gazebo/Black</material>
+  <mu1 value="200.0"/>
+  <mu2 value="100.0"/>
+  <kp value="10000000.0" />
+  <kd value="1.0" />
+  <material>Gazebo/Grey</material>
 </gazebo>
 <gazebo reference="wheel_3">
-    <material>Gazebo/Black</material>
+  <mu1 value="200.0"/>
+  <mu2 value="100.0"/>
+  <kp value="10000000.0" />
+  <kd value="1.0" />
+  <material>Gazebo/Grey</material>
 </gazebo>
 <gazebo reference="wheel_4">
-    <material>Gazebo/Black</material>
-</gazebo>
+  <mu1 value="200.0"/>
+  <mu2 value="100.0"/>
+  <kp value="10000000.0" />
+  <kd value="1.0" />
+  <material>Gazebo/Grey</material></gazebo>
   <!-- Gazebo plugin for ROS Control -->
   <gazebo>
