Commit message: now on rails :)

File: my_robot/urdf/my_robot.urdf.xacro (robot description, xacro)
@@ -4,6 +4,9 @@
   <xacro:property name="width" value="1" />
   <xacro:property name="height" value="0.5" />
-  <xacro:property name="length_wheel" value="0.2" />
-  <xacro:property name="radius_wheel" value="0.2" />
+  <xacro:property name="length_wheel_disc" value="0.01" />
+  <xacro:property name="radius_wheel_disc" value="0.15" />
+  <xacro:property name="length_wheel" value="0.11" />
+  <xacro:property name="radius_wheel" value="0.12" />
+  <xacro:property name="wheel_offset" value="0.505" />
   <xacro:macro name="default_inertial" params="mass">
     <inertial>
@@ -86,11 +89,14 @@
     <visual>
             <geometry>
-                <cylinder length="${length_wheel}" radius="${radius_wheel}"/>
+                <cylinder length="${length_wheel_disc}" radius="${radius_wheel_disc}"/>
             </geometry>
         <origin rpy="0 0 0" xyz="0 0 0"/>
-        <material name="black">
-            <color rgba="0 0 0 1"/>
-        </material>
     </visual>
+    <visual>
+      <geometry>
+          <cylinder length="${length_wheel}" radius="${radius_wheel}"/>
+      </geometry>
+      <origin rpy="0 0 0" xyz="0 0 0.055"/>
+</visual>
     <collision>
         <geometry>
@@ -103,11 +109,34 @@
   <visual>
           <geometry>
+              <cylinder length="${length_wheel_disc}" radius="${radius_wheel_disc}"/>
+          </geometry>
+      <origin rpy="0 0 0" xyz="0 0 0"/>
+  </visual>
+  <visual>
+    <geometry>
+        <cylinder length="${length_wheel}" radius="${radius_wheel}"/>
+    </geometry>
+    <origin rpy="0 0 0" xyz="0 0 -0.055"/>
+</visual>
+  <collision>
+      <geometry>
               <cylinder length="${length_wheel}" radius="${radius_wheel}"/>
+      </geometry>
+  </collision>
+  <xacro:default_inertial mass="3"/>
+</link>
+<link name="wheel_3">
+  <visual>
+          <geometry>
+              <cylinder length="${length_wheel_disc}" radius="${radius_wheel_disc}"/>
           </geometry>
       <origin rpy="0 0 0" xyz="0 0 0"/>
-      <material name="black">
-          <color rgba="0 0 0 1"/>
-      </material>
-  </visual>
+  </visual>
+  <visual>
+    <geometry>
+        <cylinder length="${length_wheel}" radius="${radius_wheel}"/>
+    </geometry>
+    <origin rpy="0 0 0" xyz="0 0 0.055"/>
+</visual>
   <collision>
       <geometry>
@@ -117,31 +146,17 @@
   <xacro:default_inertial mass="3"/>
 </link>
-<link name="wheel_3">
+<link name="wheel_4">
   <visual>
           <geometry>
-              <cylinder length="${length_wheel}" radius="${radius_wheel}"/>
+              <cylinder length="${length_wheel_disc}" radius="${radius_wheel_disc}"/>
           </geometry>
       <origin rpy="0 0 0" xyz="0 0 0"/>
-      <material name="black">
-          <color rgba="0 0 0 1"/>
-      </material>
-  </visual>
-  <collision>
-      <geometry>
-              <cylinder length="${length_wheel}" radius="${radius_wheel}"/>
-      </geometry>
-  </collision>
-  <xacro:default_inertial mass="3"/>
-</link>
-<link name="wheel_4">
-  <visual>
-          <geometry>
-              <cylinder length="${length_wheel}" radius="${radius_wheel}"/>
-          </geometry>
-      <origin rpy="0 0 0" xyz="0 0 0"/>
-      <material name="black">
-          <color rgba="0 0 0 1"/>
-      </material>
-  </visual>
+  </visual>
+  <visual>
+    <geometry>
+        <cylinder length="${length_wheel}" radius="${radius_wheel}"/>
+    </geometry>
+    <origin rpy="0 0 0" xyz="0 0 -0.055"/>
+</visual>
   <collision>
       <geometry>
@@ -179,5 +194,5 @@
     <parent link="base_link"/>
     <child link="wheel_1"/>
-    <origin rpy="0 -1.5707 0" xyz="0.6 0.4 0"/>
+    <origin rpy="0 1.5707 0" xyz="${wheel_offset} 0.4 0"/>
     <axis xyz="0 0 1" />
   </joint>
@@ -185,5 +200,5 @@
     <parent link="base_link"/>
     <child link="wheel_2"/>
-    <origin rpy="0 -1.5707 0" xyz="-0.6 0.4 0"/>
+    <origin rpy="0 1.5707 0" xyz="${-wheel_offset} 0.4 0"/>
     <axis xyz="0 0 1" />
   </joint>
@@ -191,5 +206,5 @@
     <parent link="base_link"/>
     <child link="wheel_3"/>
-    <origin rpy="0 -1.5707 0" xyz="0.6 -0.4 0"/>
+    <origin rpy="0 1.5707 0" xyz="${wheel_offset} -0.4 0"/>
     <axis xyz="0 0 1" />
   </joint>
@@ -197,5 +212,5 @@
     <parent link="base_link"/>
     <child link="wheel_4"/>
-    <origin rpy="0 -1.5707 0" xyz="-0.6 -0.4 0"/>
+    <origin rpy="0 1.5707 0" xyz="${-wheel_offset} -0.4 0"/>
     <axis xyz="0 0 1" />
   </joint>
@@ -251,5 +266,5 @@
   <kp value="10000000.0" />
   <kd value="1.0" />
-  <material>Gazebo/Grey</material>
+  <material>Gazebo/Yellow</material>
 </gazebo>
 <gazebo reference="wheel_2">
@@ -258,5 +273,5 @@
   <kp value="10000000.0" />
   <kd value="1.0" />
-  <material>Gazebo/Grey</material>
+  <material>Gazebo/Yellow</material>
 </gazebo>
 <gazebo reference="wheel_3">
@@ -265,5 +280,5 @@
   <kp value="10000000.0" />
   <kd value="1.0" />
-  <material>Gazebo/Grey</material>
+  <material>Gazebo/Yellow</material>
 </gazebo>
 <gazebo reference="wheel_4">
@@ -272,5 +287,5 @@
   <kp value="10000000.0" />
   <kd value="1.0" />
-  <material>Gazebo/Grey</material></gazebo>
+  <material>Gazebo/Yellow</material></gazebo>
   <!-- Gazebo plugin for ROS Control -->
   <gazebo>

Commit message: Add files via upload

File: my_robot/urdf/my_robot.urdf.xacro (robot description, xacro)
@@ -183,4 +183,32 @@
   <xacro:default_inertial mass="0.1"/>
 </link>
+<link name="laserscan_link">
+  <visual>
+    <geometry>
+      <box size="0.1 0.1 0.1"/>
+    </geometry>
+    <origin rpy="0 0 0" xyz="0 0 0"/>
+  </visual>
+  <collision>
+    <geometry>
+      <box size="0.1 0.1 0.1"/>
+    </geometry>
+  </collision>
+  <xacro:default_inertial mass="0.1"/>
+</link>
+<link name="camera_link">
+  <visual>
+    <geometry>
+      <box size="0.1 0.1 0.1"/>
+    </geometry>
+    <origin rpy="0 0 0" xyz="0 0 0"/>
+  </visual>
+  <collision>
+    <geometry>
+      <box size="0.1 0.1 0.1"/>
+    </geometry>
+  </collision>
+  <xacro:default_inertial mass="0.1"/>
+</link>
   <joint name="my_robot_base" type="prismatic">
     <origin rpy="0 0 0" xyz="0 0 0"/>
@@ -219,4 +247,16 @@
     <child link="imu_link"/>
     <origin rpy="0.0 0.0 0.0" xyz="0.0 0.0 0.175"/>
+    <axis xyz="0 0 1" />
+  </joint>
+  <joint name="base_to_laserscan" type="continuous">
+    <parent link="base_link"/>
+    <child link="laserscan_link"/>
+    <origin rpy="0.0 0.0 ${pi}" xyz="0.0 0.2 0.175"/>
+    <axis xyz="0 0 1" />
+  </joint>
+  <joint name="base_to_camera" type="continuous">
+    <parent link="base_link"/>
+    <child link="camera_link"/>
+    <origin rpy="0.0 0.0 ${pi/2}" xyz="0.2 0.2 0.175"/>
     <axis xyz="0 0 1" />
   </joint>
@@ -316,3 +356,96 @@
     </sensor>
   </gazebo>
+    <!-- Gazebo plugin for laser scan sensor-->
+  <gazebo reference="laserscan_link">
+    <mu1>0.2</mu1>
+    <mu2>0.2</mu2>
+    <material>Gazebo/Orange</material>
+  </gazebo>
+<gazebo reference="laserscan_link">
+    <sensor type="gpu_ray" name="head_hokuyo_sensor">
+      <pose>0 0 0 0 0 0</pose>
+      <visualize>false</visualize>
+      <update_rate>40</update_rate>
+      <ray>
+        <scan>
+          <horizontal>
+            <samples>720</samples>
+            <resolution>1</resolution>
+            <min_angle>-1.570796</min_angle>
+            <max_angle>1.570796</max_angle>
+          </horizontal>
+        </scan>
+        <range>
+          <min>0.10</min>
+          <max>30.0</max>
+          <resolution>0.01</resolution>
+        </range>
+        <noise>
+          <type>gaussian</type>
+          <!-- Noise parameters based on published spec for Hokuyo laser
+               achieving "+-30mm" accuracy at range < 10m.  A mean of 0.0m and
+               stddev of 0.01m will put 99.7% of samples within 0.03m of the true
+               reading. -->
+          <mean>0.0</mean>
+          <stddev>0.01</stddev>
+        </noise>
+      </ray>
+      <plugin name="gazebo_ros_head_hokuyo_controller" filename="libgazebo_ros_gpu_laser.so">
+        <topicName>/rrbot/laser/scan</topicName>
+        <frameName>hokuyo_link</frameName>
+      </plugin>
+    </sensor>
+  </gazebo>
+  <!-- camera -->
+   <gazebo reference="camera_link">
+    <mu1>0.2</mu1>
+    <mu2>0.2</mu2>
+    <material>Gazebo/Yellow</material>
+  </gazebo>
+  <gazebo reference="camera_link">
+    <sensor type="camera" name="camera1">
+      <update_rate>30.0</update_rate>
+      <camera name="head">
+        <horizontal_fov>1.3962634</horizontal_fov>
+        <image>
+          <width>800</width>
+          <height>800</height>
+          <format>R8G8B8</format>
+        </image>
+        <clip>
+          <near>0.02</near>
+          <far>300</far>
+        </clip>
+        <noise>
+          <type>gaussian</type>
+          <!-- Noise is sampled independently per pixel on each frame.
+               That pixel's noise value is added to each of its color
+               channels, which at that point lie in the range [0,1]. -->
+          <mean>0.0</mean>
+          <stddev>0.007</stddev>
+        </noise>
+      </camera>
+      <plugin name="camera_controller" filename="libgazebo_ros_camera.so">
+        <alwaysOn>true</alwaysOn>
+        <updateRate>0.0</updateRate>
+        <cameraName>rrbot/camera1</cameraName>
+        <imageTopicName>image_raw</imageTopicName>
+        <cameraInfoTopicName>camera_info</cameraInfoTopicName>
+        <frameName>camera_link_optical</frameName>
+        <!-- setting hackBaseline to anything but 0.0 will cause a misalignment
+            between the gazebo sensor image and the frame it is supposed to
+            be attached to -->
+        <hackBaseline>0.0</hackBaseline>
+        <distortionK1>0.0</distortionK1>
+        <distortionK2>0.0</distortionK2>
+        <distortionK3>0.0</distortionK3>
+        <distortionT1>0.0</distortionT1>
+        <distortionT2>0.0</distortionT2>
+        <CxPrime>0</CxPrime>
+        <Cx>0.0</Cx>
+        <Cy>0.0</Cy>
+        <focalLength>0.0</focalLength>
+      </plugin>
+    </sensor>
+  </gazebo>
 </robot>

Commit message: add collision, change PID val

File: my_robot/urdf/my_robot.urdf.xacro (robot description, xacro)
@@ -13,5 +13,8 @@
       <origin rpy="0.0 0 0" xyz="0 0 0"/>
       <mass value="${mass}" />
-      <inertia ixx="0.0" ixy="0.0" ixz="0.0" iyy="1.0" iyz="0.0" izz="0.0" />
+      <!--<inertia ixx="0.0" ixy="0.0" ixz="0.0" iyy="1.0" iyz="0.0" izz="0.0" />-->
+      <inertia ixx="1.0" ixy="0.0" ixz="0.0"
+               iyy="1.0" iyz="0.0"
+               izz="1.0" />
     </inertial>
   </xacro:macro>
@@ -88,19 +91,26 @@
   <link name="wheel_1">
     <visual>
-            <geometry>
-                <cylinder length="${length_wheel_disc}" radius="${radius_wheel_disc}"/>
-            </geometry>
-        <origin rpy="0 0 0" xyz="0 0 0"/>
+      <geometry>
+        <cylinder length="${length_wheel_disc}" radius="${radius_wheel_disc}"/>
+      </geometry>
+      <origin rpy="0 0 0" xyz="0 0 0"/>
     </visual>
     <visual>
       <geometry>
-          <cylinder length="${length_wheel}" radius="${radius_wheel}"/>
+        <cylinder length="${length_wheel}" radius="${radius_wheel}"/>
       </geometry>
       <origin rpy="0 0 0" xyz="0 0 0.055"/>
-</visual>
+    </visual>
     <collision>
-        <geometry>
-                <cylinder length="${length_wheel}" radius="${radius_wheel}"/>
-        </geometry>
+      <geometry>
+        <cylinder length="${length_wheel_disc}" radius="${radius_wheel_disc}"/>
+      </geometry>
+      <origin rpy="0 0 0" xyz="0 0 0"/>
+    </collision>
+    <collision>
+      <geometry>
+        <cylinder length="${length_wheel}" radius="${radius_wheel}"/>
+      </geometry>
+      <origin rpy="0 0 0" xyz="0 0 0.055"/>
     </collision>
     <xacro:default_inertial mass="3"/>
@@ -108,19 +118,26 @@
 <link name="wheel_2">
   <visual>
-          <geometry>
-              <cylinder length="${length_wheel_disc}" radius="${radius_wheel_disc}"/>
-          </geometry>
-      <origin rpy="0 0 0" xyz="0 0 0"/>
-  </visual>
-  <visual>
-    <geometry>
-        <cylinder length="${length_wheel}" radius="${radius_wheel}"/>
+    <geometry>
+      <cylinder length="${length_wheel_disc}" radius="${radius_wheel_disc}"/>
+    </geometry>
+    <origin rpy="0 0 0" xyz="0 0 0"/>
+  </visual>
+  <collision>
+    <geometry>
+      <cylinder length="${length_wheel}" radius="${radius_wheel}"/>
     </geometry>
     <origin rpy="0 0 0" xyz="0 0 -0.055"/>
-</visual>
-  <collision>
-      <geometry>
-              <cylinder length="${length_wheel}" radius="${radius_wheel}"/>
-      </geometry>
+  </collision>
+  <visual>
+    <geometry>
+      <cylinder length="${length_wheel}" radius="${radius_wheel}"/>
+    </geometry>
+    <origin rpy="0 0 0" xyz="0 0 -0.055"/>
+  </visual>
+  <collision>
+    <geometry>
+      <cylinder length="${length_wheel_disc}" radius="${radius_wheel_disc}"/>
+    </geometry>
+    <origin rpy="0 0 0" xyz="0 0 0"/>
   </collision>
   <xacro:default_inertial mass="3"/>
@@ -128,19 +145,26 @@
 <link name="wheel_3">
   <visual>
-          <geometry>
-              <cylinder length="${length_wheel_disc}" radius="${radius_wheel_disc}"/>
-          </geometry>
-      <origin rpy="0 0 0" xyz="0 0 0"/>
-  </visual>
-  <visual>
-    <geometry>
-        <cylinder length="${length_wheel}" radius="${radius_wheel}"/>
+    <geometry>
+      <cylinder length="${length_wheel_disc}" radius="${radius_wheel_disc}"/>
+    </geometry>
+    <origin rpy="0 0 0" xyz="0 0 0"/>
+  </visual>
+  <collision>
+    <geometry>
+      <cylinder length="${length_wheel}" radius="${radius_wheel}"/>
     </geometry>
     <origin rpy="0 0 0" xyz="0 0 0.055"/>
-</visual>
-  <collision>
-      <geometry>
-              <cylinder length="${length_wheel}" radius="${radius_wheel}"/>
-      </geometry>
+  </collision>
+  <visual>
+    <geometry>
+      <cylinder length="${length_wheel}" radius="${radius_wheel}"/>
+    </geometry>
+    <origin rpy="0 0 0" xyz="0 0 0.055"/>
+  </visual>
+  <collision>
+    <geometry>
+      <cylinder length="${length_wheel_disc}" radius="${radius_wheel_disc}"/>
+    </geometry>
+    <origin rpy="0 0 0" xyz="0 0 0"/>
   </collision>
   <xacro:default_inertial mass="3"/>
@@ -148,19 +172,26 @@
 <link name="wheel_4">
   <visual>
-          <geometry>
-              <cylinder length="${length_wheel_disc}" radius="${radius_wheel_disc}"/>
-          </geometry>
-      <origin rpy="0 0 0" xyz="0 0 0"/>
-  </visual>
-  <visual>
-    <geometry>
-        <cylinder length="${length_wheel}" radius="${radius_wheel}"/>
+    <geometry>
+      <cylinder length="${length_wheel_disc}" radius="${radius_wheel_disc}"/>
+    </geometry>
+    <origin rpy="0 0 0" xyz="0 0 0"/>
+  </visual>
+  <collision>
+    <geometry>
+      <cylinder length="${length_wheel}" radius="${radius_wheel}"/>
     </geometry>
     <origin rpy="0 0 0" xyz="0 0 -0.055"/>
-</visual>
-  <collision>
-      <geometry>
-              <cylinder length="${length_wheel}" radius="${radius_wheel}"/>
-      </geometry>
+  </collision>
+  <visual>
+    <geometry>
+      <cylinder length="${length_wheel}" radius="${radius_wheel}"/>
+    </geometry>
+    <origin rpy="0 0 0" xyz="0 0 -0.055"/>
+  </visual>
+  <collision>
+    <geometry>
+      <cylinder length="${length_wheel_disc}" radius="${radius_wheel_disc}"/>
+    </geometry>
+    <origin rpy="0 0 0" xyz="0 0 0"/>
   </collision>
   <xacro:default_inertial mass="3"/>

Commit message: Added GPS sensor

File: my_robot/urdf/my_robot.urdf.xacro (robot description, xacro)
@@ -214,4 +214,21 @@
   <xacro:default_inertial mass="0.1"/>
 </link>
+<link name="gps_link">
+  <visual>
+    <geometry>
+      <box size="0.1 0.1 0.1"/>
+    </geometry>
+    <origin rpy="0 0 0" xyz="0 0 0"/>
+    <material name="black">
+          <color rgba="0 0 0 1"/>
+    </material>
+  </visual>
+  <collision>
+    <geometry>
+      <box size="0.1 0.1 0.1"/>
+    </geometry>
+  </collision>
+  <xacro:default_inertial mass="0.1"/>
+</link>
 <link name="laserscan_link">
   <visual>
@@ -278,4 +295,10 @@
     <child link="imu_link"/>
     <origin rpy="0.0 0.0 0.0" xyz="0.0 0.0 0.175"/>
+    <axis xyz="0 0 1" />
+  </joint>
+  <joint name="base_to_gps" type="continuous">
+    <parent link="base_link"/>
+    <child link="gps_link"/>
+    <origin rpy="0.0 0.0 0.0" xyz="0.0 -0.2 0.175"/>
     <axis xyz="0 0 1" />
   </joint>
@@ -387,4 +410,61 @@
     </sensor>
   </gazebo>
+  <!-- Gazebo plugin for GPS
+  <gazebo reference="gps_link">
+    <gravity>true</gravity>
+    <sensor name="imu_sensor" type="imu">
+      <always_on>true</always_on>
+      <update_rate>40</update_rate>
+      <visualize>false</visualize>
+      <topic>__default_topic__</topic>
+      <plugin filename="libhector_gazebo_ros_gps.so" name="gps_plugin">
+        <topicName>gps</topicName>
+        <bodyName>gps_link</bodyName>
+        <updateRateHZ>50.0</updateRateHZ>
+        <gaussianNoise>0.0</gaussianNoise>
+        <xyzOffset>0 0 0</xyzOffset>
+        <rpyOffset>0 0 0</rpyOffset>
+        <frameName>gps_link</frameName>
+        <initialOrientationAsReference>false</initialOrientationAsReference>
+      </plugin>
+      <pose>0 0 0 0 0 0</pose>
+    </sensor>
+  </gazebo> -->
+  <!-- Plugin for GPS sensor -->
+  <gazebo reference="gps_link">
+    <material>Gazebo/White</material>
+  </gazebo>
+  <gazebo>
+      <plugin name="gps_sim" filename="libhector_gazebo_ros_gps.so">
+        <updateRate>40</updateRate>
+        <!--<robotNamespace>/my_robot</robotNamespace>-->
+        <bodyName>gps_link</bodyName>
+        <!--<frameId>${properties['tf_prefix']}/${name}</frameId>-->
+        <topicName>gps</topicName>
+        <!--<accelOffset>${properties['accel_offset_x']} ${properties['accel_offset_y']} ${properties['accel_offset_z']}</accelOffset>
+        <accelDrift>${properties['accel_drift_x']} ${properties['accel_drift_y']} ${properties['accel_drift_z']}</accelDrift>
+        <accelGaussianNoise>${properties['accel_noise_x']} ${properties['accel_noise_y']} ${properties['accel_noise_z']}</accelGaussianNoise>
+        <rateOffset>${properties['rate_offset_x']} ${properties['rate_offset_y']} ${properties['rate_offset_z']}</rateOffset>
+        <rateDrift>${properties['rate_drift_x']} ${properties['rate_drift_y']} ${properties['rate_drift_z']}</rateDrift>
+        <rateGaussianNoise>${properties['rate_noise_x']} ${properties['rate_noise_y']} ${properties['rate_noise_z']}</rateGaussianNoise>
+        <yawOffset>${properties['heading_offset']}</yawOffset>
+        <yawDrift>${properties['heading_drift']}</yawDrift>
+        <yawGaussianNoise>${properties['heading_noise']}</yawGaussianNoise>-->
+      </plugin>
+    </gazebo>
+<!-- Plugin for GPS sensor
+<gazebo reference= "gps_link">
+  <controller:hector_gazebo_ros_gps name="quadrotor_gps_sim" plugin="libhector_gazebo_ros_gps.so">
+    <alwaysOn>true</alwaysOn>
+    <updateRate>40.0</updateRate>
+    <bodyName>gps_link</bodyName>
+    <topicName>gps</topicName>
+    <velocityTopicName>gps_vel</velocityTopicName>
+    <drift>0.0 0.0 0.0</drift>
+    <gaussianNoise>0.0 0.0 0.0</gaussianNoise>
+    <velocityDrift>0 0 0</velocityDrift>
+    <velocityGaussianNoise>0.0 0.0 0.0</velocityGaussianNoise>
+  </controller:hector_gazebo_ros_gps>
+</gazebo> -->
     <!-- Gazebo plugin for laser scan sensor-->
   <gazebo reference="laserscan_link">
