Commit message: 2d rail and conical wheels

File: my_robot/urdf/my_robot.urdf.xacro (robot description, xacro)
@@ -9,4 +9,6 @@
   <xacro:property name="radius_wheel" value="0.12" />
   <xacro:property name="wheel_offset" value="0.505" />
+  <xacro:property name="cone_scale" value="0.5 0.5 0.5" />
+  <xacro:property name="cone_name" value="cone_long.dae" />
   <xacro:macro name="default_inertial" params="mass">
     <inertial>
@@ -87,55 +89,31 @@
       </geometry>
     </collision>
-    <xacro:default_inertial mass="10"/>
+    <xacro:default_inertial mass="30"/>
   </link>
   <link name="wheel_1">
     <visual>
-      <geometry>
-        <cylinder length="${length_wheel_disc}" radius="${radius_wheel_disc}"/>
-      </geometry>
+        <geometry>
+          <mesh filename="package://my_robot/urdf/${cone_name}" scale="${cone_scale}"/>
+        </geometry>
       <origin rpy="0 0 0" xyz="0 0 0"/>
     </visual>
-    <visual>
-      <geometry>
-        <cylinder length="${length_wheel}" radius="${radius_wheel}"/>
-      </geometry>
-      <origin rpy="0 0 0" xyz="0 0 0.055"/>
-    </visual>
     <collision>
       <geometry>
-        <cylinder length="${length_wheel_disc}" radius="${radius_wheel_disc}"/>
+        <mesh filename="package://my_robot/urdf/${cone_name}" scale="${cone_scale}"/>
       </geometry>
       <origin rpy="0 0 0" xyz="0 0 0"/>
     </collision>
-    <collision>
-      <geometry>
-        <cylinder length="${length_wheel}" radius="${radius_wheel}"/>
-      </geometry>
-      <origin rpy="0 0 0" xyz="0 0 0.055"/>
-    </collision>
     <xacro:default_inertial mass="3"/>
 </link>
-<link name="wheel_2">
-  <visual>
-    <geometry>
-      <cylinder length="${length_wheel_disc}" radius="${radius_wheel_disc}"/>
-    </geometry>
-    <origin rpy="0 0 0" xyz="0 0 0"/>
-  </visual>
-  <collision>
-    <geometry>
-      <cylinder length="${length_wheel}" radius="${radius_wheel}"/>
-    </geometry>
-    <origin rpy="0 0 0" xyz="0 0 -0.055"/>
-  </collision>
-  <visual>
-    <geometry>
-      <cylinder length="${length_wheel}" radius="${radius_wheel}"/>
-    </geometry>
-    <origin rpy="0 0 0" xyz="0 0 -0.055"/>
-  </visual>
-  <collision>
-    <geometry>
-      <cylinder length="${length_wheel_disc}" radius="${radius_wheel_disc}"/>
+  <link name="wheel_2">
+    <visual>
+      <geometry>
+        <mesh filename="package://my_robot/urdf/${cone_name}" scale="${cone_scale}"/>
+      </geometry>
+    <origin rpy="0 0 0" xyz="0 0 0"/>
+  </visual>
+  <collision>
+    <geometry>
+      <mesh filename="package://my_robot/urdf/${cone_name}" scale="${cone_scale}"/>
     </geometry>
     <origin rpy="0 0 0" xyz="0 0 0"/>
@@ -146,54 +124,30 @@
   <visual>
     <geometry>
-      <cylinder length="${length_wheel_disc}" radius="${radius_wheel_disc}"/>
-    </geometry>
-    <origin rpy="0 0 0" xyz="0 0 0"/>
-  </visual>
-  <collision>
-    <geometry>
-      <cylinder length="${length_wheel}" radius="${radius_wheel}"/>
-    </geometry>
-    <origin rpy="0 0 0" xyz="0 0 0.055"/>
-  </collision>
-  <visual>
-    <geometry>
-      <cylinder length="${length_wheel}" radius="${radius_wheel}"/>
-    </geometry>
-    <origin rpy="0 0 0" xyz="0 0 0.055"/>
-  </visual>
-  <collision>
-    <geometry>
-      <cylinder length="${length_wheel_disc}" radius="${radius_wheel_disc}"/>
-    </geometry>
-    <origin rpy="0 0 0" xyz="0 0 0"/>
-  </collision>
-  <xacro:default_inertial mass="3"/>
+      <mesh filename="package://my_robot/urdf/${cone_name}" scale="${cone_scale}"/>
+    </geometry>
+  <origin rpy="0 0 0" xyz="0 0 0"/>
+</visual>
+<collision>
+  <geometry>
+    <mesh filename="package://my_robot/urdf/${cone_name}" scale="${cone_scale}"/>
+  </geometry>
+  <origin rpy="0 0 0" xyz="0 0 0"/>
+</collision>
+<xacro:default_inertial mass="3"/>
 </link>
 <link name="wheel_4">
   <visual>
     <geometry>
-      <cylinder length="${length_wheel_disc}" radius="${radius_wheel_disc}"/>
-    </geometry>
-    <origin rpy="0 0 0" xyz="0 0 0"/>
-  </visual>
-  <collision>
-    <geometry>
-      <cylinder length="${length_wheel}" radius="${radius_wheel}"/>
-    </geometry>
-    <origin rpy="0 0 0" xyz="0 0 -0.055"/>
-  </collision>
-  <visual>
-    <geometry>
-      <cylinder length="${length_wheel}" radius="${radius_wheel}"/>
-    </geometry>
-    <origin rpy="0 0 0" xyz="0 0 -0.055"/>
-  </visual>
-  <collision>
-    <geometry>
-      <cylinder length="${length_wheel_disc}" radius="${radius_wheel_disc}"/>
-    </geometry>
-    <origin rpy="0 0 0" xyz="0 0 0"/>
-  </collision>
-  <xacro:default_inertial mass="3"/>
+      <mesh filename="package://my_robot/urdf/${cone_name}" scale="${cone_scale}"/>
+    </geometry>
+  <origin rpy="0 0 0" xyz="0 0 0"/>
+</visual>
+<collision>
+  <geometry>
+    <mesh filename="package://my_robot/urdf/${cone_name}" scale="${cone_scale}"/>
+  </geometry>
+  <origin rpy="0 0 0" xyz="0 0 0"/>
+</collision>
+<xacro:default_inertial mass="3"/>
 </link>
 <link name="imu_link">
@@ -276,5 +230,5 @@
     <parent link="base_link"/>
     <child link="wheel_2"/>
-    <origin rpy="0 1.5707 0" xyz="${-wheel_offset} 0.4 0"/>
+    <origin rpy="0 4.7121 0" xyz="${-wheel_offset} 0.4 0"/>
     <axis xyz="0 0 1" />
   </joint>
@@ -288,5 +242,5 @@
     <parent link="base_link"/>
     <child link="wheel_4"/>
-    <origin rpy="0 1.5707 0" xyz="${-wheel_offset} -0.4 0"/>
+    <origin rpy="0 4.7121 0" xyz="${-wheel_offset} -0.4 0"/>
     <axis xyz="0 0 1" />
   </joint>

Commit message: changed sensor joints to fixed, they liked to spin around now that the robot tilts in corners

File: my_robot/urdf/my_robot.urdf.xacro (robot description, xacro)
@@ -188,11 +188,11 @@
   <visual>
     <geometry>
-      <box size="0.1 0.1 0.1"/>
-    </geometry>
-    <origin rpy="0 0 0" xyz="0 0 0"/>
-  </visual>
-  <collision>
-    <geometry>
-      <box size="0.1 0.1 0.1"/>
+      <box size="0.1 0.1 0.2"/>
+    </geometry>
+    <origin rpy="0 0 0" xyz="0 0 0"/>
+  </visual>
+  <collision>
+    <geometry>
+      <box size="0.1 0.1 0.2"/>
     </geometry>
   </collision>
@@ -245,5 +245,5 @@
     <axis xyz="0 0 1" />
   </joint>
-  <joint name="base_to_imu" type="continuous">
+  <joint name="base_to_imu" type="fixed">
     <parent link="base_link"/>
     <child link="imu_link"/>
@@ -251,5 +251,5 @@
     <axis xyz="0 0 1" />
   </joint>
-  <joint name="base_to_gps" type="continuous">
+  <joint name="base_to_gps" type="fixed">
     <parent link="base_link"/>
     <child link="gps_link"/>
@@ -257,11 +257,11 @@
     <axis xyz="0 0 1" />
   </joint>
-  <joint name="base_to_laserscan" type="continuous">
+  <joint name="base_to_laserscan" type="fixed">
     <parent link="base_link"/>
     <child link="laserscan_link"/>
-    <origin rpy="0.0 0.0 ${pi}" xyz="0.0 0.2 0.175"/>
-    <axis xyz="0 0 1" />
-  </joint>
-  <joint name="base_to_camera" type="continuous">
+    <origin rpy="0.0 0.0 ${pi}" xyz="0.0 0.2 0.375"/>
+    <axis xyz="0 0 1" />
+  </joint>
+  <joint name="base_to_camera" type="fixed">
     <parent link="base_link"/>
     <child link="camera_link"/>

Commit message: changed the visual size of the laser-scanner. Updated its refreshrate from 40 to 200 to allow for increased vehicle speed

File: my_robot/urdf/my_robot.urdf.xacro (robot description, xacro)
@@ -188,11 +188,11 @@
   <visual>
     <geometry>
-      <box size="0.1 0.1 0.2"/>
-    </geometry>
-    <origin rpy="0 0 0" xyz="0 0 0"/>
-  </visual>
-  <collision>
-    <geometry>
-      <box size="0.1 0.1 0.2"/>
+      <box size="0.05 0.05 0.4"/>
+    </geometry>
+    <origin rpy="0 0 0" xyz="0 0 0"/>
+  </visual>
+  <collision>
+    <geometry>
+      <box size="0.05 0.05 0.4"/>
     </geometry>
   </collision>
@@ -260,5 +260,5 @@
     <parent link="base_link"/>
     <child link="laserscan_link"/>
-    <origin rpy="0.0 0.0 ${pi}" xyz="0.0 0.2 0.375"/>
+    <origin rpy="0.0 0.0 ${pi}" xyz="0.0 0.2 0.300"/>
     <axis xyz="0 0 1" />
   </joint>
@@ -405,5 +405,5 @@
       <pose>0 0 0 0 0 0</pose>
       <visualize>true</visualize>
-      <update_rate>40</update_rate>
+      <update_rate>200</update_rate>
       <ray>
         <scan>

Commit message: modify the length of robot and size of wheel

File: my_robot/urdf/my_robot.urdf.xacro (robot description, xacro)
@@ -1,5 +1,5 @@
 <?xml version="1.0"?>
 <robot xmlns:xacro="http://www.ros.org/wiki/xacro" name="my_robot">
-  <xacro:property name="length" value="1" />
+  <xacro:property name="length" value="1.21" />
   <xacro:property name="width" value="1" />
   <xacro:property name="height" value="0.5" />
@@ -8,7 +8,7 @@
   <xacro:property name="length_wheel" value="0.11" />
   <xacro:property name="radius_wheel" value="0.12" />
-  <xacro:property name="wheel_offset" value="0.505" />
+  <xacro:property name="wheel_offset" value="0.61" />
   <xacro:property name="cone_scale" value="0.5 0.5 0.5" />
-  <xacro:property name="cone_name" value="cone_long.dae" />
+  <xacro:property name="cone_name" value="cone.dae" />
   <xacro:macro name="default_inertial" params="mass">
     <inertial>

Commit message: simplify startup of my_robot to one file, add packages to CMakeLists files

File: my_robot/urdf/my_robot.urdf.xacro (robot description, xacro)
@@ -21,8 +21,22 @@
     </inertial>
   </xacro:macro>
-<!--
-  <link name="my_robot_xpart">
-    <visual>
-      <origin rpy="0 0 0" xyz="0 0 ${height/2}"/>
+  <link name="base_footprint">
+    <visual>
+      <origin rpy="0 0 0" xyz="0 0 0"/>
+      <geometry>
+        <box size="0 0 0"/>
+      </geometry>
+    </visual>
+    <collision>
+      <origin rpy="0 0 0" xyz="0 0 0"/>
+      <geometry>
+        <box size="0 0 0"/>
+      </geometry>
+    </collision>
+    <xacro:default_inertial mass="0.1"/>
+  </link>
+  <link name="base_link">
+    <visual>
+      <origin rpy="0 0 0" xyz="0 0 0"/>
       <geometry>
         <box size="${length} ${width} ${height/2}"/>
@@ -30,71 +44,62 @@
     </visual>
     <collision>
-      <origin rpy="0 0 0" xyz="0 0 ${height/2}"/>
+      <origin rpy="0 0 0" xyz="0 0 0"/>
       <geometry>
         <box size="${length} ${width} ${height/2}"/>
       </geometry>
     </collision>
-    <xacro:default_inertial mass="10"/>
-  </link>
-  <gazebo reference="my_robot_xpart">
-    <mu1>10.0</mu1>
-    <mu2>10.0</mu2>
-    <material> Gazebo/GreyTransparent</material>
-  </gazebo>
-  <joint name="my_robot_x" type="prismatic">
+    <xacro:default_inertial mass="30"/>
+  </link>
+  <link name="wheel_1">
+    <visual>
+      <geometry>
+        <mesh filename="package://my_robot/urdf/${cone_name}" scale="${cone_scale}"/>
+      </geometry>
+      <origin rpy="0 0 0" xyz="0 0 0"/>
+    </visual>
+    <collision>
+      <geometry>
+        <mesh filename="package://my_robot/urdf/${cone_name}" scale="${cone_scale}"/>
+      </geometry>
+      <origin rpy="0 0 0" xyz="0 0 0"/>
+    </collision>
+    <xacro:default_inertial mass="3"/>
+  </link>
+  <link name="wheel_2">
+    <visual>
+      <geometry>
+        <mesh filename="package://my_robot/urdf/${cone_name}" scale="${cone_scale}"/>
+      </geometry>
+      <origin rpy="0 0 0" xyz="0 0 0"/>
+    </visual>
+    <collision>
+      <geometry>
+        <mesh filename="package://my_robot/urdf/${cone_name}" scale="${cone_scale}"/>
+      </geometry>
+      <origin rpy="0 0 0" xyz="0 0 0"/>
+    </collision>
+    <xacro:default_inertial mass="3"/>
+  </link>
+  <link name="wheel_3">
+    <visual>
+      <geometry>
+        <mesh filename="package://my_robot/urdf/${cone_name}" scale="${cone_scale}"/>
+      </geometry>
+      <origin rpy="0 0 0" xyz="0 0 0"/>
+    </visual>
+    <collision>
+      <geometry>
+        <mesh filename="package://my_robot/urdf/${cone_name}" scale="${cone_scale}"/>
+      </geometry>
+      <origin rpy="0 0 0" xyz="0 0 0"/>
+    </collision>
+    <xacro:default_inertial mass="3"/>
+  </link>
+  <link name="wheel_4">
+    <visual>
+      <geometry>
+        <mesh filename="package://my_robot/urdf/${cone_name}" scale="${cone_scale}"/>
+      </geometry>
     <origin rpy="0 0 0" xyz="0 0 0"/>
-    <parent link="world"/>
-    <child link="my_robot_xpart"/>
-    <axis xyz="1 0 0"/>
-    <dynamics damping="0" friction="0"/>
-    <limit effort="10000" lower="-50.0" upper="50.0" velocity="1"/>
-  </joint>
-  <transmission name="tran1">
-    <type>transmission_interface/SimpleTransmission</type>
-    <joint name="my_robot_x">
-      <hardwareInterface>EffortJointInterface</hardwareInterface>
-    </joint>
-    <actuator name="motor1">
-      <hardwareInterface>EffortJointInterface</hardwareInterface>
-      <mechanicalReduction>1</mechanicalReduction>
-    </actuator>
-  </transmission>
--->
-<link name="base_footprint">
-  <visual>
-    <origin rpy="0 0 0" xyz="0 0 0"/>
-    <geometry>
-      <box size="0 0 0"/>
-    </geometry>
-  </visual>
-  <collision>
-    <origin rpy="0 0 0" xyz="0 0 0"/>
-    <geometry>
-      <box size="0 0 0"/>
-    </geometry>
-  </collision>
-  <xacro:default_inertial mass="0.1"/>
-</link>
-  <link name="base_link">
-    <visual>
-      <origin rpy="0 0 0" xyz="0 0 0"/>
-      <geometry>
-        <box size="${length} ${width} ${height/2}"/>
-      </geometry>
-    </visual>
-    <collision>
-      <origin rpy="0 0 0" xyz="0 0 0"/>
-      <geometry>
-        <box size="${length} ${width} ${height/2}"/>
-      </geometry>
-    </collision>
-    <xacro:default_inertial mass="30"/>
-  </link>
-  <link name="wheel_1">
-    <visual>
-        <geometry>
-          <mesh filename="package://my_robot/urdf/${cone_name}" scale="${cone_scale}"/>
-        </geometry>
-      <origin rpy="0 0 0" xyz="0 0 0"/>
     </visual>
     <collision>
@@ -105,112 +110,53 @@
     </collision>
     <xacro:default_inertial mass="3"/>
-</link>
-  <link name="wheel_2">
-    <visual>
-      <geometry>
-        <mesh filename="package://my_robot/urdf/${cone_name}" scale="${cone_scale}"/>
-      </geometry>
-    <origin rpy="0 0 0" xyz="0 0 0"/>
-  </visual>
-  <collision>
-    <geometry>
-      <mesh filename="package://my_robot/urdf/${cone_name}" scale="${cone_scale}"/>
-    </geometry>
-    <origin rpy="0 0 0" xyz="0 0 0"/>
-  </collision>
-  <xacro:default_inertial mass="3"/>
-</link>
-<link name="wheel_3">
-  <visual>
-    <geometry>
-      <mesh filename="package://my_robot/urdf/${cone_name}" scale="${cone_scale}"/>
-    </geometry>
-  <origin rpy="0 0 0" xyz="0 0 0"/>
-</visual>
-<collision>
-  <geometry>
-    <mesh filename="package://my_robot/urdf/${cone_name}" scale="${cone_scale}"/>
-  </geometry>
-  <origin rpy="0 0 0" xyz="0 0 0"/>
-</collision>
-<xacro:default_inertial mass="3"/>
-</link>
-<link name="wheel_4">
-  <visual>
-    <geometry>
-      <mesh filename="package://my_robot/urdf/${cone_name}" scale="${cone_scale}"/>
-    </geometry>
-  <origin rpy="0 0 0" xyz="0 0 0"/>
-</visual>
-<collision>
-  <geometry>
-    <mesh filename="package://my_robot/urdf/${cone_name}" scale="${cone_scale}"/>
-  </geometry>
-  <origin rpy="0 0 0" xyz="0 0 0"/>
-</collision>
-<xacro:default_inertial mass="3"/>
-</link>
-<link name="imu_link">
-  <visual>
-    <geometry>
-      <box size="0.1 0.1 0.1"/>
-    </geometry>
-    <origin rpy="0 0 0" xyz="0 0 0"/>
-    <material name="black">
-          <color rgba="0 0 0 1"/>
-    </material>
-  </visual>
-  <collision>
-    <geometry>
-      <box size="0.1 0.1 0.1"/>
-    </geometry>
-  </collision>
-  <xacro:default_inertial mass="0.1"/>
-</link>
-<link name="gps_link">
-  <visual>
-    <geometry>
-      <box size="0.1 0.1 0.1"/>
-    </geometry>
-    <origin rpy="0 0 0" xyz="0 0 0"/>
-    <material name="black">
-          <color rgba="0 0 0 1"/>
-    </material>
-  </visual>
-  <collision>
-    <geometry>
-      <box size="0.1 0.1 0.1"/>
-    </geometry>
-  </collision>
-  <xacro:default_inertial mass="0.1"/>
-</link>
-<link name="laserscan_link">
-  <visual>
-    <geometry>
-      <box size="0.05 0.05 0.4"/>
-    </geometry>
-    <origin rpy="0 0 0" xyz="0 0 0"/>
-  </visual>
-  <collision>
-    <geometry>
-      <box size="0.05 0.05 0.4"/>
-    </geometry>
-  </collision>
-  <xacro:default_inertial mass="0.1"/>
-</link>
-<link name="camera_link">
-  <visual>
-    <geometry>
-      <box size="0.1 0.1 0.1"/>
-    </geometry>
-    <origin rpy="0 0 0" xyz="0 0 0"/>
-  </visual>
-  <collision>
-    <geometry>
-      <box size="0.1 0.1 0.1"/>
-    </geometry>
-  </collision>
-  <xacro:default_inertial mass="0.1"/>
-</link>
+  </link>
+  <link name="imu_link">
+    <visual>
+      <geometry>
+        <box size="0.1 0.1 0.1"/>
+      </geometry>
+      <origin rpy="0 0 0" xyz="0 0 0"/>
+      <material name="black">
+        <color rgba="0 0 0 1"/>
+      </material>
+    </visual>
+    <collision>
+      <geometry>
+        <box size="0.1 0.1 0.1"/>
+      </geometry>
+    </collision>
+    <xacro:default_inertial mass="0.1"/>
+  </link>
+  <link name="gps_link">
+    <visual>
+      <geometry>
+        <box size="0.1 0.1 0.1"/>
+      </geometry>
+      <origin rpy="0 0 0" xyz="0 0 0"/>
+      <material name="black">
+        <color rgba="0 0 0 1"/>
+      </material>
+    </visual>
+    <collision>
+      <geometry>
+        <box size="0.1 0.1 0.1"/>
+      </geometry>
+    </collision>
+    <xacro:default_inertial mass="0.1"/>
+  </link>
+  <link name="laserscan_link">
+    <visual>
+      <geometry>
+        <box size="0.05 0.05 0.4"/>
+      </geometry>
+      <origin rpy="0 0 0" xyz="0 0 0"/>
+    </visual>
+    <collision>
+      <geometry>
+        <box size="0.05 0.05 0.4"/>
+      </geometry>
+    </collision>
+    <xacro:default_inertial mass="0.1"/>
+  </link>
   <joint name="my_robot_base" type="prismatic">
     <origin rpy="0 0 0" xyz="0 0 0"/>
@@ -263,82 +209,61 @@
     <axis xyz="0 0 1" />
   </joint>
-  <joint name="base_to_camera" type="fixed">
-    <parent link="base_link"/>
-    <child link="camera_link"/>
-    <origin rpy="0.0 0.0 ${pi/2}" xyz="0.2 0.2 0.175"/>
-    <axis xyz="0 0 1" />
-  </joint>
-  <transmission name="tran2">
+  <transmission name="transmission_wheel_1">
     <type>transmission_interface/SimpleTransmission</type>
-    <joint name="my_robot_base">
-      <hardwareInterface>EffortJointInterface</hardwareInterface>
+    <joint name="base_to_wheel1">
+      <hardwareInterface>hardware_interface/EffortJointInterface</hardwareInterface>
     </joint>
-    <actuator name="motor2">
-      <hardwareInterface>EffortJointInterface</hardwareInterface>
+    <actuator name="motor_wheel_1">
+      <hardwareInterface>hardware_interface/EffortJointInterface</hardwareInterface>
       <mechanicalReduction>1</mechanicalReduction>
     </actuator>
   </transmission>
-  <transmission name="transmission_wheel_1">
+  <transmission name="transmission_wheel_2">
     <type>transmission_interface/SimpleTransmission</type>
-    <joint name="base_to_wheel1">
-        <hardwareInterface>hardware_interface/EffortJointInterface</hardwareInterface>
+    <joint name="base_to_wheel2">
+      <hardwareInterface>hardware_interface/EffortJointInterface</hardwareInterface>
     </joint>
-    <actuator name="motor_wheel_1">
-        <hardwareInterface>hardware_interface/EffortJointInterface</hardwareInterface>
-        <mechanicalReduction>1</mechanicalReduction>
-    </actuator>
-</transmission>
-<transmission name="transmission_wheel_2">
-  <type>transmission_interface/SimpleTransmission</type>
-  <joint name="base_to_wheel2">
-      <hardwareInterface>hardware_interface/EffortJointInterface</hardwareInterface>
-  </joint>
-  <actuator name="motor_wheel_2">
+    <actuator name="motor_wheel_2">
       <hardwareInterface>hardware_interface/EffortJointInterface</hardwareInterface>
       <mechanicalReduction>1</mechanicalReduction>
-  </actuator>
-</transmission>
-<!--
-  <joint name="entity" type="fixed">
-    <origin rpy="0 0 0" xyz="0 0 0"/>
-    <parent link="my_robot_xpart"/>
-    <child link="my_robot_ypart"/>
-  </joint>-->
-<gazebo reference="base_link">
+    </actuator>
+  </transmission>
+  <gazebo reference="base_link">
     <material>Gazebo/Blue</material>
     <gravity>1</gravity>
-</gazebo>
-<gazebo reference="wheel_1">
-  <mu1 value="200.0"/>
-  <mu2 value="100.0"/>
-  <kp value="10000000.0" />
-  <kd value="1.0" />
-  <material>Gazebo/Yellow</material>
-</gazebo>
-<gazebo reference="wheel_2">
-  <mu1 value="200.0"/>
-  <mu2 value="100.0"/>
-  <kp value="10000000.0" />
-  <kd value="1.0" />
-  <material>Gazebo/Yellow</material>
-</gazebo>
-<gazebo reference="wheel_3">
-  <mu1 value="200.0"/>
-  <mu2 value="100.0"/>
-  <kp value="10000000.0" />
-  <kd value="1.0" />
-  <material>Gazebo/Yellow</material>
-</gazebo>
-<gazebo reference="wheel_4">
-  <mu1 value="200.0"/>
-  <mu2 value="100.0"/>
-  <kp value="10000000.0" />
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
Commit message: full overhaul of laser (x wonky in turns)

File: my_robot/urdf/my_robot.urdf.xacro (robot description, xacro)
@@ -206,5 +206,5 @@
     <parent link="base_link"/>
     <child link="laserscan_link"/>
-    <origin rpy="0.0 0.0 ${pi}" xyz="0.0 0.2 0.300"/>
+    <origin rpy="0.0 0.0 ${pi}" xyz="0.0 0.2 0.800"/>
     <axis xyz="0 0 1" />
   </joint>
@@ -328,5 +328,5 @@
         <range>
           <min>0.10</min>
-          <max>35.0</max>
+          <max>40.0</max>
           <resolution>0.01</resolution>
         </range>
